File: hardware/boopbox-proto/audio_max98357a.kicad_sch (KiCad schematic)
At the start: 3 parts, among them U3 MAX98357A breakout

Commit message: Settle on MAX98357A audio stage in KiCad schematic
Drop the PCM5102A + MAX98306 option sheet (kept in history at 1c76144),
mark GPIO12 reserved for the amp SD pin, update sheet notes and title
blocks, and ignore KiCad lock/backup files. ERC: 0 violations.

Co-Authored-By: Claude Opus 5.5 <noreply@anthropic.com>
Other:
- note added: "AUDIO NOTES - VIN from 5V (Feather USB pin) for full output; 3.3V works but is much quieter. - C1 sits right at the amp's VIN/GND on the breadboard to stop brownout resets on loud peaks. - GAIN unconnected = 9 dB. SD unconnected = (L+R)/2 mono mix via the board's on-board resistor. - Do NOT tie SD straight to a 3.3V GPIO: a solid high selects LEFT channel only. If you want GPIO mute, check the MA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"
- note removed: "OPTION A NOTES - VIN from 5V (Feather USB pin) for full output; 3.3V works but is much quieter. - C1 sits right at the amp's VIN/GND on the breadboard to stop brownout resets on loud peaks. - GAIN unconnected = 9 dB. SD unconnected = (L+R)/2 mono mix via the board's on-board resistor. - Do NOT tie SD straight to a 3.3V GPIO: a solid high selects LEFT channel only. If you want GPIO mute, check the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"
- title: Audio option A: MAX98357A -> Audio: MAX98357A
Changed lines of the file:
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@@
 (kicad_sch (version 20250114) (generator "eeschema") (generator_version "9.0")
 (paper "USLetter")
-(title_block (title "Audio option A: MAX98357A") (date "2026-10-12") (rev "A") (company "BoopBox") (comment 1 "Single board: I2S in, speaker out (recommended)"))
+(title_block (title "Audio: MAX98357A") (date "2026-10-17") (rev "B") (company "BoopBox") (comment 1 "Single board: I2S in, speaker out"))
 (symbol (lib_id "boopbox-proto:MAX98357A_Breakout") (at 101.6 88.9 0) (unit 1) (exclude_from_sim no) (in_bom yes) (on_board yes) (dnp no)
   (property "Reference" "U3" (at 101.6 77.47 0) (effects (font (size 1.27 1.27))))
@@
 )
 (text "C1: place at U3 VIN/GND" (exclude_from_sim no) (at 81.28 119.38 0) (effects (font (size 1.27 1.27)) (justify left top)))
-(text "OPTION A NOTES\n- VIN from 5V (Feather USB pin) for full output; 3.3V works but is much quieter.\n- C1 sits right at the amp's VIN/GND on the breadboard to stop brownout resets on loud peaks.\n- GAIN unconnected = 9 dB. SD unconnected = (L+R)/2 mono mix via the board's on-board resistor.\n- Do NOT tie SD straight to a 3.3V GPIO: a solid high selects LEFT channel only. If you want\n  GPIO mute, check the MAX98357A datasheet SD_MODE thresholds and size a series resistor first.\n- Speaker goes across SPK+ / SPK-. Outputs are bridge-tied: never connect either one to GND." (exclude_from_sim no) (at 127 119.38 0) (effects (font (size 1.27 1.27)) (justify left top)))
+(text "AUDIO NOTES\n- VIN from 5V (Feather USB pin) for full output; 3.3V works but is much quieter.\n- C1 sits right at the amp's VIN/GND on the breadboard to stop brownout resets on loud peaks.\n- GAIN unconnected = 9 dB. SD unconnected = (L+R)/2 mono mix via the board's on-board resistor.\n- Do NOT tie SD straight to a 3.3V GPIO: a solid high selects LEFT channel only. If you want\n  GPIO mute, check the MAX98357A datasheet SD_MODE thresholds and size a series resistor first.\n- Speaker goes across SPK+ / SPK-. Outputs are bridge-tied: never connect either one to GND." (exclude_from_sim no) (at 127 119.38 0) (effects (font (size 1.27 1.27)) (justify left top)))
 (embedded_fonts no)
 )
