File: hardware/boopbox-proto/boopbox-proto.kicad_sch (KiCad schematic)
At the start: 2 parts, among them U1 Feather ESP32-S3 (4MB/2MB PSR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, U2 PN532 NFC (I2C mode)

Commit message: Settle on MAX98357A audio stage in KiCad schematic
Drop the PCM5102A + MAX98306 option sheet (kept in history at 1c76144),
mark GPIO12 reserved for the amp SD pin, update sheet notes and title
blocks, and ignore KiCad lock/backup files. ERC: 0 violations.

Co-Authored-By: Claude Opus 5.5 <noreply@anthropic.com>
Connections:
- net AMP_SD: no longer names the net of U1.21 (D12/GPIO12)
- no-connect marks 19 -> 20
Other:
- sheet Audio option A: MAX98357A renamed Audio: MAX98357A
- removed sheet Audio option B: PCM5102A + MAX98306
- note added: "Audio stage:"
- note added: "BREADBOARD NOTES 1. PN532: set the DIP switch to I2C before powering up. Feather has 5k pull-ups on SDA/SCL; the PN532 board's own pull-ups in parallel are fine. 2. Avoid GPIO7 (STEMMA QT / I2C power enable), GPIO21 + GPIO33 (NeoPixel). 3. USB pin = 5V only while powered from USB-C. On battery it is unpowered: amp would need BAT. 4. Audio: MAX98357A (I2S DAC + amp) on the sheet below. The PCM5102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"
- note removed: "BREADBOARD NOTES 1. PN532: set the DIP switch to I2C before powering up. Feather has 5k pull-ups on SDA/SCL; the PN532 board's own pull-ups in parallel are fine. 2. Avoid GPIO7 (STEMMA QT / I2C power enable), GPIO21 + GPIO33 (NeoPixel). 3. USB pin = 5V only while powered from USB-C. On battery it is unpowered: amp would need BAT. 4. Audio stage: build ONE of the two sheets below. They share the I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"
- note removed: "Pick ONE audio stage:"
Changed lines of the file:
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@@
 (kicad_sch (version 20250114) (generator "eeschema") (generator_version "9.0")
 (paper "USLetter")
-(title_block (title "BoopBox breadboard prototype") (date "2026-10-12") (rev "A") (company "BoopBox") (comment 1 "Feather ESP32-S3 + PN532 + audio stage (pick ONE)"))
+(title_block (title "BoopBox breadboard prototype") (date "2026-10-17") (rev "B") (company "BoopBox") (comment 1 "Feather ESP32-S3 + PN532 + MAX98357A audio"))
 (symbol (lib_id "boopbox-proto:Feather_ESP32-S3_N4R2") (at 101.6 96.52 0) (unit 1) (exclude_from_sim no) (in_bom yes) (on_board yes) (dnp no)
   (property "Reference" "U1" (at 101.6 73.66 0) (effects (font (size 1.27 1.27))))
@@
 )
 (no_connect (at 124.46 85.09))
-(wire (pts (xy 124.46 87.63) (xy 129.54 87.63)) (stroke (width 0) (type default)))
-(global_label "AMP_SD" (shape output) (at 129.54 87.63 0) (fields_autoplaced yes) (effects (font (size 1.27 1.27)) (justify left)))
+(no_connect (at 124.46 87.63))
 (wire (pts (xy 124.46 90.17) (xy 129.54 90.17)) (stroke (width 0) (type default)))
 (global_label "I2S_DIN" (shape output) (at 129.54 90.17 0) (fields_autoplaced yes) (effects (font (size 1.27 1.27)) (justify left)))
@@
 )
 (text "PWR_FLAG: tells ERC the GND net is driven (Feather GND pin is passive)." (exclude_from_sim no) (at 55.88 129.54 0) (effects (font (size 1.27 1.27)) (justify left top)))
-(text "BREADBOARD NOTES\n1. PN532: set the DIP switch to I2C before powering up. Feather has 5k pull-ups on SDA/SCL;\n   the PN532 board's own pull-ups in parallel are fine.\n2. Avoid GPIO7 (STEMMA QT / I2C power enable), GPIO21 + GPIO33 (NeoPixel).\n3. USB pin = 5V only while powered from USB-C. On battery it is unpowered: amp would need BAT.\n4. Audio stage: build ONE of the two sheets below. They share the I2S_* / AMP_SD nets,\n   so ERC and netlists show both connected at once. That is documentation, not a circuit.\n5. ESPHome: i2s_audio lrclk=GPIO10, bclk=GPIO9, dout=GPIO11; i2c sda=GPIO3, scl=GPIO4." (exclude_from_sim no) (at 152.4 99.06 0) (effects (font (size 1.27 1.27)) (justify left top)))
+(text "BREADBOARD NOTES\n1. PN532: set the DIP switch to I2C before powering up. Feather has 5k pull-ups on SDA/SCL;\n   the PN532 board's own pull-ups in parallel are fine.\n2. Avoid GPIO7 (STEMMA QT / I2C power enable), GPIO21 + GPIO33 (NeoPixel).\n3. USB pin = 5V only while powered from USB-C. On battery it is unpowered: amp would need BAT.\n4. Audio: MAX98357A (I2S DAC + amp) on the sheet below. The PCM5102A + MAX98306 option was\n   dropped; it lives in git history (commit 1c76144).\n   GPIO12 is reserved for the MAX98357A SD pin (mute/sleep); not wired yet (SD floats = L+R mix).\n5. ESPHome: i2s_audio lrclk=GPIO10, bclk=GPIO9, dout=GPIO11; i2c sda=GPIO3, scl=GPIO4." (exclude_from_sim no) (at 152.4 99.06 0) (effects (font (size 1.27 1.27)) (justify left top)))
 (sheet (at 165.1 134.62) (size 63.5 7.62) (exclude_from_sim no) (in_bom yes) (on_board yes) (dnp no) (stroke (width 0.1524) (type solid)) (fill (color 0 0 0 0.0000))
-  (property "Sheetname" "Audio option A: MAX98357A" (at 165.1 133.92 0) (effects (font (size 1.27 1.27)) (justify left bottom)))
+  (property "Sheetname" "Audio: MAX98357A" (at 165.1 133.92 0) (effects (font (size 1.27 1.27)) (justify left bottom)))
   (property "Sheetfile" "audio_max98357a.kicad_sch" (at 165.1 142.84 0) (effects (font (size 1.27 1.27)) (justify left top)))
   (instances (project "boopbox-proto" (path "/cf3ae905-5af5-44db-b9d8-9bea9527c364" (page "2"))))
 )
-(sheet (at 165.1 152.4) (size 63.5 7.62) (exclude_from_sim no) (in_bom yes) (on_board yes) (dnp no) (stroke (width 0.1524) (type solid)) (fill (color 0 0 0 0.0000))
-  (property "Sheetname" "Audio option B: PCM5102A + MAX98306" (at 165.1 151.7 0) (effects (font (size 1.27 1.27)) (justify left bottom)))
-  (property "Sheetfile" "audio_pcm5102a_max98306.kicad_sch" (at 165.1 160.62 0) (effects (font (size 1.27 1.27)) (justify left top)))
-  (instances (project "boopbox-proto" (path "/cf3ae905-5af5-44db-b9d8-9bea9527c364" (page "3"))))
-)
-(text "Pick ONE audio stage:" (exclude_from_sim no) (at 165.1 124.46 0) (effects (font (size 1.5 1.5)) (justify left top)))
+(text "Audio stage:" (exclude_from_sim no) (at 165.1 124.46 0) (effects (font (size 1.5 1.5)) (justify left top)))
 (sheet_instances (path "/" (page "1")))
 (embedded_fonts no)
